File: Interposer to PCIEx16.kicad_sch (KiCad schematic)
At the start: 27 parts, among them U1 BuckBoostIC, U2 PGOOD, U3 5v_Regulator, U4 +12V, U5 VIN, U6 GND

Commit message: Add files via upload
V0.2
Parts:
- removed C1, C7: 22uf, FW 16 Components:22uf 25V, symbol FW 16 Components:22uf
- removed C3, C5: ~, FW 16 Components:1210 capacitor, symbol FW 16 Components:1210_capacitor
- removed J1: ~, FW 16 Components:PCI-Ex16, symbol FW 16 Components:PCI-Ex16
- removed J2: ~, FW 16 Components:FW 16 Interposer DB, symbol FW 16 Components:Interposer_DB_
- removed L1: ~, FW 16 Components:3.3uH, symbol FW 16 Components:3.3uH
- removed R11: 10k, FW 16 Components:0603, symbol FW 16 Components:0603
- removed U1: BuckBoostIC, FW 16 Components:BuckBoostIC, symbol FW 16 Components:AOZ2261AQI-15
- removed U2: PGOOD, FW 16 Components:PAD, symbol FW 16 Components:PAD
- removed U3: 5v_Regulator, FW 16 Components:5v Regulator, symbol FW 16 Components:5v_Regulator
- removed U4: +12V, FW 16 Components:PAD, symbol FW 16 Components:PAD
- removed U5: VIN, FW 16 Components:PAD, symbol FW 16 Components:PAD
- removed U6: GND, FW 16 Components:PAD, symbol FW 16 Components:PAD
- added C1: 1.0uf, FW 16 Components:1210 capacitor, symbol FW 16 Components:1210_capacitor
- added C3, C5, C7: 100uf, FW 16 Components:25SVPF100M, symbol FW 16 Components:25SVPF100M
- added J1: ~, FW 16 Components:FW 16 Interposer DB, symbol FW 16 Components:Interposer_DB_
- added J2: ~, FW 16 Components:PCI-Ex16, symbol FW 16 Components:PCI-Ex16
- added J3, J4, J5: ~, FW 16 Components:TestPad, symbol FW 16 Components:TestPad
- added J6, J7, J8, J9: ~, FW 16 Components:PowerTHT, symbol FW 16 Components:PowerTHT
- added L1: WE-XHMA_1090, FW 16 Components:WE-XHMA_1090, symbol FW 16 Components:WE-XHMA_1090
- added R12: 10k, FW 16 Components:0603, symbol FW 16 Components:0603
- added R13: 10, FW 16 Components:0603, symbol FW 16 Components:0603
- added U3: BD9F800MUX-ZE2, FW 16 Components:VQFN11_ROM, symbol FW 16 Components:BD9F800MUX-ZE2
- C4: value ~ -> .1uf
- C6: value .01uf -> .1uf
- R10: value 10k -> 10
- R6: value 200k -> 47.5k
- R7: value 10k -> 100k
- R8: value 30k -> 10k
- R9: value 140k -> 10k
Connections:
- net +12V: now also C6.2, R10.2, R6.1, C7.1, J2.A2 (+12V), J2.A3 (+12V), J2.B1 (+12V), J2.B2 (+12V), J2.B3 (+12V), J8.1, L1.2; no longer C4.1, R9.2
- net +3.3V: now also J1.PA4 (3.3V_ALW), J1.PA5 (3.3V_ALW), J1.PB4 (3.3V_ALW), J1.PB5 (3.3V_ALW), J2.A10 (+3.3V), J2.A9 (+3.3V), J2.B10 (+3.3V_AUX), J2.B8 (+3.3V)
- net +5V: now also J1.PK7 (5V_ALW), J1.PK8 (5V_ALW), J1.PL7 (5V_ALW), J1.PL8 (5V_ALW)
- net GND: now also C4.1, C6.1, R1.1, R2.1, R4.2, R5.2, R8.2, C1.2, C3.2, C5.2, C7.2, J1.PA3 (GND), J1.PA6 (GND), J1.PB3 (GND), J1.PB6 (GND), J1.PC6 (GND), J1.PD1 (GND), J1.PD2 (GND), J1.PD6 (GND), J1.PE1 (GND), J1.PE2 (GND), J1.PE3 (GND), J1.PE6 (GND), J1.PF1 (GND), J1.PF6 (GND), J1.PG6 (GND), J1.PH3 (GND), J1.PH6 (GND), J1.PH7 (GND), J1.PH8 (GND), J1.PJ6 (GND), J1.PJ7 (GND), J1.PJ8 (GND), J1.PK4 (GND), J1.PK6 (GND), J1.PL3 (GND), J1.PL6 (GND), J1.SB2 (GND), J1.SB7 (GND), J1.SC1 (GND), J1.SC3 (GND), J1.SC6 (GND), J1.SC8 (GND), J1.SE2 (GND), J1.SE7 (GND), J1.SF1 (GND), J1.SF3 (GND), J1.SF6 (GND), J1.SF8 (GND), J1.SH2 (GND), J1.SH7 (GND), J1.SJ1 (GND), J1.SJ3 (GND), J1.SJ6 (GND), J1.SJ8 (GND), J2.A12 (GND), J2.A15 (GND), J2.A18 (GND), J2.A20 (GND), J2.A23 (GND), J2.A24 (GND), J2.A27 (GND), J2.A28 (GND), J2.A31 (GND), J2.A34 (GND), J2.A37 (GND), J2.A38 (GND), J2.A4 (GND), J2.A41 (GND), J2.A42 (GND), J2.A45 (GND), J2.A46 (GND), J2.A49 (GND), J2.A51 (GND), J2.A52 (PEX_RX8P), J2.A54 (GND), J2.A55 (GND), J2.A58 (GND), J2.A59 (GND), J2.A62 (GND), J2.A63 (GND), J2.A66 (GND), J2.A67 (GND), J2.A70 (GND), J2.A71 (GND), J2.A74 (GND), J2.A75 (GND), J2.A78 (GND), J2.A79 (GND), J2.A82 (GND), J2.B13 (GND), J2.B18 (GND), J2.B21 (GND), J2.B22 (GND), J2.B25 (GND), J2.B26 (GND), J2.B29 (GND), J2.B32 (GND), J2.B35 (GND), J2.B36 (GND), J2.B39 (GND), J2.B4 (GND), J2.B40 (GND), J2.B43 (GND), J2.B44 (GND), J2.B47 (GND), J2.B49 (GND), J2.B52 (GND), J2.B53 (GND), J2.B56 (GND), J2.B57 (GND), J2.B60 (GND), J2.B61 (GND), J2.B64 (GND), J2.B65 (GND), J2.B68 (GND), J2.B69 (GND), J2.B7 (GND), J2.B72 (GND), J2.B73 (GND), J2.B76 (GND), J2.B77 (GND), J2.B80 (GND), J7.1, J9.1, R12.2, U3.10 (PGND), U3.7 (GND); no longer C4.2, C6.2, R1.2, R10.1, R2.2, R4.1, R5.1, R7.1
- net H_RX0N: now also J1.SG8 (PEX_TX0N), J2.A17 (PEX_RX0N)
- net H_RX0P: now also J1.SH8 (PEX_TX0P), J2.A16 (PEX_RX0P)
- net H_RX1N: now also J1.SK8 (PEX_TX1N), J2.A22 (PEX_RX1N)
- net H_RX1P: now also J1.SL8 (PEX_TX1P), J2.A21 (PEX_RX1P)
- net H_RX2N: now also J1.SH6 (PEX_TX2N), J2.A26 (PEX_RX2N)
- net H_RX2P: now also J1.SG6 (PEX_TX2P), J2.A25 (PEX_RX2P)
- net H_RX3N: now also J1.SK6 (PEX_TX3N), J2.A30 (PEX_RX3N)
- net H_RX3P: now also J1.SL6 (PEX_TX3P), J2.A29 (PEX_RX3P)
- net H_RX4N: now also J1.SL3 (PEX_TX4N), J2.A36 (PEX_RX4N)
- net H_RX4P: now also J1.SK3 (PEX_TX4P), J2.A35 (PEX_RX4P)
- net H_RX5N: now also J1.SG3 (PEX_TX5N), J2.A40 (PEX_RX5N)
- net H_RX5P: now also J1.SH3 (PEX_TX5P), J2.A39 (PEX_RX5P)
- net H_RX6N: now also J1.SL1 (PEX_TX6N), J2.A44 (PEX_RX6N)
- net H_RX6P: now also J1.SK1 (PEX_TX6P), J2.A43 (PEX_RX6P)
- net H_RX7N: now also J1.SG1 (PEX_TX7N), J2.A48 (PEX_RX7N)
- net H_RX7P: now also J1.SH1 (PEX_TX7P), J2.A47 (PEX_RX7P)
- net H_TX0N: now also J1.SD8 (PEX_RX0N), J2.B15 (PEX_TX0N)
- net H_TX0P: now also J1.SE8 (PEX_RX0P), J2.B14 (PEX_TX0P)
- net H_TX1N: now also J1.SA8 (PEX_RX1N), J2.B20 (PEX_TX1N)
- net H_TX1P: now also J1.SB8 (PEX_RX1P), J2.B19 (PEX_TX1P)
- net H_TX2N: now also J1.SD6 (PEX_RX2N), J2.B24 (PEX_TX2N)
- net H_TX2P: now also J1.SE6 (PEX_RX2P), J2.B23 (PEX_TX2P)
- net H_TX3N: now also J1.SA6 (PEX_RX3N), J2.B28 (PEX_TX3N)
- net H_TX3P: now also J1.SB6 (PEX_RX3P), J2.B27 (PEX_TX3P)
- net H_TX4N: now also J1.SB3 (PEX_RX4N), J2.B34 (PEX_TX4N)
- net H_TX4P: now also J1.SA3 (PEX_RX4P), J2.B33 (PEX_TX4P)
- net H_TX5N: now also J1.SE3 (PEX_RX5N), J2.B38 (PEX_TX5N)
- net H_TX5P: now also J1.SD3 (PEX_RX5P), J2.B37 (PEX_TX5P)
- net H_TX6N: now also J1.SB1 (PEX_RX6N), J2.B42 (PEX_TX6N)
- net H_TX6P: now also J1.SA1 (PEX_RX6P), J2.B41 (PEX_TX6P)
- net H_TX7N: now also J1.SD1 (PEX_RX7N), J2.B46 (PEX_TX7N)
- net H_TX7P: now also J1.SE1 (PEX_RX7P), J2.B45 (PEX_TX7P)
- net PERST_RST: now also J1.SA5 (PEX_RST#), J2.A11 (PERST#)
- net PRSNT: now also J2.A1 (PRNST#1), J2.B48 (PRSNT2#)
- net REFCLK+: now also J1.SC2 (PEX_REFCLK), J2.A13 (REFCLK+)
- net REFCLK-: now also J1.SD2 (PEX_REFCLK#), J2.A14 (REFCLK-)
- net VIN: now also C4.2, C3.1, C5.1, J1.PA7 (VSYS_GPU), J1.PA8 (VSYS_GPU), J1.PB7 (VSYS_GPU), J1.PB8 (VSYS_GPU), J1.PC7 (VSYS_GPU), J1.PC8 (VSYS_GPU), J1.PD7 (VSYS_GPU), J1.PD8 (VSYS_GPU), J1.PE7 (VSYS_GPU), J1.PE8 (VSYS_GPU), J1.PF7 (VSYS_GPU), J1.PF8 (VSYS_GPU), J1.PG7 (VSYS_GPU), J1.PG8 (VSYS_GPU), J5.1, J6.1, U3.11 (EN), U3.8 (VIN); no longer R6.1, R8.2
- net at C2.1: now also U3.1 (BOOT)
- net at R6.2: now also R7.1
- net at R3.1: now also J2.A5 (TCK)
- net EN: no longer names the net of R7.2, R8.1
- net EN: now also J4.1, R13.2
- net FB: no longer names the net of R9.1
- net FB: now also J3.1, U3.2 (PGD); no longer R10.2
- net LX renamed SW
- net SW: now also L1.1, U3.9 (SW)
- new net: R10.1, U3.3 (VOUT)
- new net: R13.1, U3.5 (FB)
- new net: J1.SA4 (PEX_CLK_REQ#), R1.2
- new net: J2.A6 (TDI), R5.1
- new net: J2.A8 (TMS), R4.1
- new net: J2.B9 (TRST#), R2.2
- new net: R12.1, U3.4 (FREQ)
- new net: J1.PA1 (VADP_GPU), J1.PA2 (VADP_GPU), J1.PB1 (VADP_GPU), J1.PB2 (VADP_GPU), J1.PC1 (VADP_GPU), J1.PC2 (VADP_GPU)
- new net VREG: C1.1, R9.2, U3.6 (VREG)
